Commit message: Add an example with a horizontal passive joint

File: gazebo_ros2_control_demos/urdf/test_arm_effort.xacro.urdf (robot description, URDF)
Before this commit: robot pendulum on cart, 2 links, 3 joints
Links:
- removed link slideBar
Joints:
- removed joint slider_to_cart
- joint cart_to_pendulum: origin xyz=0.0 0.35 0.0 rpy=0 0.1 0 -> xyz=0.0 0.0 0.2 rpy=1.57 0 0
- joint world_to_base: child slideBar -> cart; limit (none) -> lower=-15 upper=15 effort=1000.0 velocity=30
